Commit message: 添加了新的功能

File: learn_ws/src/simplebb/xacro/my_move.urdf.xacro (robot description, xacro)
@@ -29,6 +29,14 @@
             <rightRearJoint>b_r_j</rightRearJoint>
             <odometryRate>1000</odometryRate>
-            <robotBaseFrame>base_link</robotBaseFrame>
+            <robotBaseFrame>base_footprint</robotBaseFrame>
             <broadcastTF>1</broadcastTF>
+            <cmdVelTimeOut>0.25</cmdVelTimeOut>
+            <publishOdometryTf>0</publishOdometryTf>
+            <yaw_velocity_p_gain>1.0</yaw_velocity_p_gain>
+            <x_velocity_p_gain>15.0</x_velocity_p_gain>
+            <y_velocity_p_gain>15.0</y_velocity_p_gain>
+            <max_x_velocity>0.6</max_x_velocity>
+            <max_y_velocity>0.6</max_y_velocity>
+            <max_yaw_velocity>0.5</max_yaw_velocity>
         </plugin>
     </gazebo>

File: learn_ws/src/simplebb/xacro/simplebb.urdf.xacro (robot description, xacro)
@@ -1,5 +1,5 @@
 <robot name="simplebb"
     xmlns:xacro="http://www.ros.org/wiki/xacro">
-    <!-- <link name="base_footprint">
+    <link name="base_footprint">
         <visual>
             <geometry>
@@ -7,10 +7,12 @@
             </geometry>
         </visual>
-    </link>  -->
+    </link>
     <link name="base_link">
         <inertial>
             <origin xyz="0 0 0.1981" rpy="0 0 0" />
             <mass value="7.1499" />
-            <inertia ixx="0.19541" ixy="-5.5057E-18" ixz="4.3095E-17" iyy="0.24546" iyz="-1.468E-17" izz="0.41766" />
+            <inertia ixx="0.19541" ixy="0" ixz="0"
+                     iyy="0.24546" iyz="0"
+                     izz="0.41766" />
         </inertial>
         <visual>
@@ -30,9 +32,9 @@
         </collision>
     </link>
-    <!-- <joint name="base_link2base_footprint" type="fixed">
+    <joint name="base_link2base_footprint" type="fixed">
         <parent link="base_footprint" />
         <child link="base_link" />
-        <origin xyz="0 0 0.14842" />
-    </joint> -->
+        <origin xyz="0 0 0.00006" />
+    </joint>
     <xacro:mc_wheel link_name="b_r" axis_y="1" joint_x="-1" joint_y="-1"/>
     <xacro:mc_wheel link_name="b_l" axis_y="-1" joint_x="-1" joint_y="1"/>

File: learn_ws/src/simplebb/xacro/wheel.urdf.xacro (robot description, xacro)
@@ -6,5 +6,7 @@
                 <origin xyz="1.305E-06 ${-0.0001226*axis_y} 4.6233E-06" rpy="0 0 0" />
                 <mass value="0.21836" />
-                <inertia ixx="0.00010444" ixy="-9.9501E-08" ixz="-1.3183E-07" iyy="0.00018522" iyz="2.8085E-08" izz="0.00010401" />
+                <inertia ixx="0.00010444" ixy="0" ixz="0"
+                         iyy="0.00018522" iyz="0"
+                         izz="0.00010401" />
             </inertial>
             <visual>
@@ -29,5 +31,5 @@
             <child link="${link_name}_l" />
             <axis xyz="0 ${axis_y} 0" />
-            <limit effort="30" velocity="17.4" />
+            <limit effort="30000000" velocity="17.4" />
         </joint>
     </xacro:macro>

Commit message: ps4_

File: learn_ws/src/simplebb/xacro/my_move.urdf.xacro (robot description, xacro)
@@ -33,10 +33,10 @@
             <cmdVelTimeOut>0.25</cmdVelTimeOut>
             <publishOdometryTf>0</publishOdometryTf>
-            <yaw_velocity_p_gain>1.0</yaw_velocity_p_gain>
-            <x_velocity_p_gain>15.0</x_velocity_p_gain>
-            <y_velocity_p_gain>15.0</y_velocity_p_gain>
-            <max_x_velocity>15</max_x_velocity>
-            <max_y_velocity>15</max_y_velocity>
-            <max_yaw_velocity>1</max_yaw_velocity>
+            <yaw_velocity_p_gain>1000.0</yaw_velocity_p_gain>
+            <x_velocity_p_gain>15000.0</x_velocity_p_gain>
+            <y_velocity_p_gain>15000.0</y_velocity_p_gain>
+            <max_x_velocity>10000000</max_x_velocity>
+            <max_y_velocity>10000000</max_y_velocity>
+            <max_yaw_velocity>1000</max_yaw_velocity>
         </plugin>
     </gazebo>

File: learn_ws/src/simplebb/xacro/my_sensors_laser.urdf.xacro (robot description, xacro)
@@ -4,5 +4,5 @@
     <sensor type="ray" name="rplidar">
       <pose>0 0 0 0 0 0</pose>
-      <visualize>true</visualize>
+      <visualize>false</visualize>
       <update_rate>15</update_rate>
       <ray>
@@ -11,6 +11,6 @@
             <samples>360</samples>
             <resolution>1</resolution>
-            <min_angle>-3</min_angle>
-            <max_angle>3</max_angle>
+            <min_angle>-3.14</min_angle>
+            <max_angle>3.141</max_angle>
           </horizontal>
         </scan>

File: learn_ws/src/simplebb/xacro/wheel.urdf.xacro (robot description, xacro)
@@ -31,5 +31,5 @@
             <child link="${link_name}_l" />
             <axis xyz="0 ${axis_y} 0" />
-            <limit effort="30000000" velocity="17.4" />
+            <limit effort="30000000000" velocity="550" />
         </joint>
     </xacro:macro>
